Commit message: Add MuJoCo config and integrate with description, not working yet

File: src/ur5_workbench_description/urdf/ur5_workbench.urdf.xacro (robot description, xacro)
@@ -2,15 +2,17 @@
 <robot name="ur5_workbench" xmlns:xacro="http://www.ros.org/wiki/xacro">
   <xacro:include filename="$(find ur5_workbench_description)/urdf/ur5_workbench_macro.xacro" />
-  <xacro:arg name="thing1_joint_limits_parameters_file" default="$(find ur5_workbench_description)/config/ur5/joint_limits.yaml"/>
-  <xacro:arg name="thing1_kinematics_parameters_file" default="$(find ur5_workbench_description)/config/ur5/default_kinematics.yaml"/>
-  <xacro:arg name="thing1_physical_parameters_file" default="$(find ur5_workbench_description)/config/ur5/physical_parameters.yaml"/>
-  <xacro:arg name="thing1_visual_parameters_file" default="$(find ur5_workbench_description)/config/ur5/visual_parameters.yaml"/>
-  <xacro:arg name="thing2_joint_limits_parameters_file" default="$(find ur5_workbench_description)/config/ur5/joint_limits.yaml"/>
-  <xacro:arg name="thing2_kinematics_parameters_file" default="$(find ur5_workbench_description)/config/ur5/default_kinematics.yaml"/>
-  <xacro:arg name="thing2_physical_parameters_file" default="$(find ur5_workbench_description)/config/ur5/physical_parameters.yaml"/>
-  <xacro:arg name="thing2_visual_parameters_file" default="$(find ur5_workbench_description)/config/ur5/visual_parameters.yaml"/>
+  <xacro:arg name="include_ros2_control" default="true"/>
+  <xacro:arg name="thing1_joint_limits_parameters_file" default="$(find ur_description)/config/ur5/joint_limits.yaml"/>
+  <xacro:arg name="thing1_kinematics_parameters_file" default="$(find ur_description)/config/ur5/default_kinematics.yaml"/>
+  <xacro:arg name="thing1_physical_parameters_file" default="$(find ur_description)/config/ur5/physical_parameters.yaml"/>
+  <xacro:arg name="thing1_visual_parameters_file" default="$(find ur_description)/config/ur5/visual_parameters.yaml"/>
+  <xacro:arg name="thing2_joint_limits_parameters_file" default="$(find ur_description)/config/ur5/joint_limits.yaml"/>
+  <xacro:arg name="thing2_kinematics_parameters_file" default="$(find ur_description)/config/ur5/default_kinematics.yaml"/>
+  <xacro:arg name="thing2_physical_parameters_file" default="$(find ur_description)/config/ur5/physical_parameters.yaml"/>
+  <xacro:arg name="thing2_visual_parameters_file" default="$(find ur_description)/config/ur5/visual_parameters.yaml"/>
   <link name="world" />
   <xacro:ur5_workbench
     parent="world"
+    include_ros2_control="$(arg include_ros2_control)"
     thing1_joint_limits_parameters_file="$(arg thing1_joint_limits_parameters_file)"
     thing1_kinematics_parameters_file="$(arg thing1_kinematics_parameters_file)"
@@ -23,4 +25,4 @@
   >
     <origin xyz="0 0 1" rpy="0 0 0" />
-  </xacro:things>
+  </xacro:ur5_workbench>
 </robot>

File: src/ur5_workbench_description/urdf/ur5_workbench_macro.xacro (robot description, xacro)
@@ -2,4 +2,7 @@
 <robot xmlns:xacro="http://www.ros.org/wiki/xacro">
   <xacro:include filename="$(find ur_description)/urdf/ur_macro.xacro" />
+  <xacro:include filename="$(find robotiq_ft_sensor_description)/urdf/robotiq_ft300.urdf.xacro" />
+  <xacro:include filename="$(find robotiq_description)/urdf/robotiq_2f_85_macro.urdf.xacro" />
+  <xacro:include filename="$(find robotiq_ft_sensor_description)/urdf/robotiq_fts.ros2_control.xacro" />
   <xacro:macro
     name="ur5_workbench"
@@ -7,4 +10,5 @@
       parent
       *origin
+      include_ros2_control:=true
       thing1_joint_limits_parameters_file
       thing1_kinematics_parameters_file
@@ -40,4 +44,21 @@
       <origin xyz="0 0 0" rpy="0 0 0" />
     </xacro:ur_robot>
+    <xacro:robotiq_ft300 parent="flange" tf_prefix="thing1_">
+      <origin xyz="0 0 0" rpy="0 0 0" />
+    </xacro:robotiq_ft300>
+    <xacro:if value="${include_ros2_control}">
+      <xacro:robotiq_fts_ros2_control
+        name="thing1_"
+        tf_prefix="thing1_"
+      />
+    </xacro:if>
+    <xacro:robotiq_gripper
+      name="thing1_robotiq_gripper"
+      parent="thing1_ft300_sensor"
+      prefix="thing1_"
+      include_ros2_control="${include_ros2_control}"
+    >
+      <origin xyz="0 0 0" rpy="0 0 0" />
+    </xacro:robotiq_gripper>
     <link name="thing2_robot_mount" />
     <joint name="thing2_robot_mount_joint" type="fixed">
@@ -57,4 +78,21 @@
       <origin xyz="0 0 0" rpy="0 0 0" />
     </xacro:ur_robot>
+    <xacro:robotiq_ft300 parent="flange" tf_prefix="thing2_">
+      <origin xyz="0 0 0" rpy="0 0 0" />
+    </xacro:robotiq_ft300>
+    <xacro:if value="${include_ros2_control}">
+      <xacro:robotiq_fts_ros2_control
+        name="thing2_"
+        tf_prefix="thing2_"
+      />
+    </xacro:if>
+    <xacro:robotiq_gripper
+      name="thing2_robotiq_gripper"
+      parent="thing2_ft300_sensor"
+      prefix="thing2_"
+      include_ros2_control="${include_ros2_control}"
+    >
+      <origin xyz="0 0 0" rpy="0 0 0" />
+    </xacro:robotiq_gripper>
   </xacro:macro>
 </robot>
