Commit message: Add tcp frame

File: src/ur5_workbench_description/urdf/thing_macro.xacro (robot description, xacro)
@@ -84,4 +84,10 @@
       />
     </xacro:if>
+    <joint name="${name}_tcp_joint" type="fixed">
+      <origin xyz="0 0 0.135" rpy="0 0 0" />
+      <parent link="${name}_robotiq_85_base_link" />
+      <child link="${name}_tcp_frame" />
+    </joint>
+    <link name="${name}_tcp_frame" />
   </xacro:macro>
 </robot>

Commit message: Lots of changes

File: src/ur5_workbench_description/urdf/thing_macro.xacro (robot description, xacro)
@@ -2,10 +2,22 @@
 <robot xmlns:xacro="http://www.ros.org/wiki/xacro">
   <xacro:include filename="$(find ur_description)/urdf/ur_macro.xacro" />
-  <xacro:include filename="$(find robotiq_ft_sensor_description)/urdf/robotiq_ft300.urdf.xacro" />
-  <xacro:include filename="$(find robotiq_description)/urdf/robotiq_2f_85_macro.urdf.xacro" />
-  <xacro:include filename="$(find robotiq_ft_sensor_description)/urdf/robotiq_fts.ros2_control.xacro" />
-  <xacro:include filename="$(find ur5_workbench_description)/urdf/camera_mount_macro.xacro" />
-  <xacro:include filename="$(find ur_robot_driver)/urdf/ur.ros2_control.xacro" />
-  <xacro:macro name="thing" params="
+  <xacro:include
+        filename="$(find robotiq_ft_sensor_description)/urdf/robotiq_ft300.urdf.xacro"
+    />
+  <xacro:include
+        filename="$(find robotiq_description)/urdf/robotiq_2f_85_macro.urdf.xacro"
+    />
+  <xacro:include
+        filename="$(find robotiq_ft_sensor_description)/urdf/robotiq_fts.ros2_control.xacro"
+    />
+  <xacro:include
+        filename="$(find ur5_workbench_description)/urdf/camera_mount_macro.xacro"
+    />
+  <xacro:include
+        filename="$(find ur_robot_driver)/urdf/ur.ros2_control.xacro"
+    />
+  <xacro:macro
+        name="thing"
+        params="
     name
     parent
@@ -17,4 +29,8 @@
     physical_parameters_file
     visual_parameters_file
+    use_fts:=true
+    fts_dev:=ttyUSB0
+    use_gripper:=true
+    gripper_com_port:='/dev/ttyUSB2'
     robot_ip:=''
     script_filename:=''
@@ -22,14 +38,15 @@
     output_recipe_filename:=''
     initial_positions:=${dict(shoulder_pan_joint=0.0,shoulder_lift_joint=-1.57,elbow_joint=0.0,wrist_1_joint=-1.57,wrist_2_joint=0.0,wrist_3_joint=0.0)}
-  ">
+  "
+    >
     <xacro:ur_robot
-      name="${name}"
-      tf_prefix="${name}_"
-      parent="${parent}"
-      joint_limits_parameters_file="${joint_limits_parameters_file}"
-      kinematics_parameters_file="${kinematics_parameters_file}"
-      physical_parameters_file="${physical_parameters_file}"
-      visual_parameters_file="${visual_parameters_file}"
-    >
+            name="${name}"
+            tf_prefix="${name}_"
+            parent="${parent}"
+            joint_limits_parameters_file="${joint_limits_parameters_file}"
+            kinematics_parameters_file="${kinematics_parameters_file}"
+            physical_parameters_file="${physical_parameters_file}"
+            visual_parameters_file="${visual_parameters_file}"
+        >
       <xacro:insert_block name="origin" />
     </xacro:ur_robot>
@@ -38,20 +55,27 @@
     </xacro:robotiq_ft300>
     <xacro:if value="${wrist_camera_model != ''}">
-      <xacro:include filename="$(find realsense2_description)/urdf/_${wrist_camera_model}.urdf.xacro" />
-      <xacro:camera_mount parent="${name}_robotiq_ft_frame_id" tf_prefix="${name}_">
+      <xacro:include
+                filename="$(find realsense2_description)/urdf/_${wrist_camera_model}.urdf.xacro"
+            />
+      <xacro:camera_mount
+                parent="${name}_robotiq_ft_frame_id"
+                tf_prefix="${name}_"
+            >
         <origin xyz="0 0 0" rpy="0 0 0" />
       </xacro:camera_mount>
-      <xacro:call macro="sensor_${wrist_camera_model}"
-        name="${name}_${wrist_camera_model}"
-        parent="${name}_camera_link"
-      >
-        <origin xyz="0 0.021 0.009" rpy="0 ${-pi/2} ${pi/2}"/>
+      <xacro:call
+                macro="sensor_${wrist_camera_model}"
+                name="${name}_${wrist_camera_model}"
+                parent="${name}_camera_link"
+            >
+        <origin xyz="0 0.021 0.009" rpy="0 ${-pi/2} ${pi/2}" />
       </xacro:call>
       <xacro:robotiq_gripper
-        name="${name}_robotiq_gripper"
-        parent="${name}_tool_link"
-        prefix="${name}_"
-        include_ros2_control="${include_ros2_control}"
-      >
+                name="${name}_robotiq_gripper"
+                parent="${name}_tool_link"
+                prefix="${name}_"
+                include_ros2_control="${include_ros2_control and use_gripper}"
+                com_port="${gripper_com_port}"
+            >
         <origin xyz="0 0 0" rpy="0 0 0" />
       </xacro:robotiq_gripper>
@@ -59,9 +83,10 @@
     <xacro:unless value="${wrist_camera_model != ''}">
       <xacro:robotiq_gripper
-        name="${name}_robotiq_gripper"
-        parent="${name}_robotiq_ft_frame_id"
-        prefix="${name}_"
-        include_ros2_control="${include_ros2_control}"
-      >
+                name="${name}_robotiq_gripper"
+                parent="${name}_robotiq_ft_frame_id"
+                prefix="${name}_"
+                include_ros2_control="${include_ros2_control and use_gripper}"
+                com_port="${gripper_com_port}"
+            >
         <origin xyz="0 0 0" rpy="0 0 0" />
       </xacro:robotiq_gripper>
@@ -69,18 +94,22 @@
     <!-- ros2_control macros -->
     <xacro:if value="${include_ros2_control}">
-      <xacro:robotiq_fts_ros2_control
-        name="${name}_"
-        tf_prefix="${name}_"
-      />
+      <xacro:if value="${use_fts}">
+        <xacro:robotiq_fts_ros2_control
+                    name="${name}_"
+                    tf_prefix="${name}_"
+                    ftdi_id="${fts_dev}"
+                />
+      </xacro:if>
       <xacro:ur_ros2_control
-        name="${name}_"
-        tf_prefix="${name}_"
-        kinematics_parameters_file="${kinematics_parameters_file}"
-        robot_ip="${robot_ip}"
-        script_filename="${script_filename}"
-        input_recipe_filename="${input_recipe_filename}"
-        output_recipe_filename="${output_recipe_filename}"
-        initial_positions="${initial_positions}"
-      />
+                name="${name}"
+                tf_prefix="${name}_"
+                kinematics_parameters_file="${kinematics_parameters_file}"
+                robot_ip="${robot_ip}"
+                script_filename="${script_filename}"
+                input_recipe_filename="${input_recipe_filename}"
+                output_recipe_filename="${output_recipe_filename}"
+                initial_positions="${initial_positions}"
+                script_sender_port="50002"
+            />
     </xacro:if>
     <joint name="${name}_tcp_joint" type="fixed">

File: src/ur5_workbench_description/urdf/ur5_workbench.urdf.xacro (robot description, xacro)
@@ -1,45 +1,87 @@
 <?xml version="1.0" ?>
 <robot name="ur5_workbench" xmlns:xacro="http://www.ros.org/wiki/xacro">
-  <xacro:include filename="$(find ur5_workbench_description)/urdf/ur5_workbench_macro.xacro" />
-  <xacro:arg name="include_ros2_control" default="false"/>
-  <xacro:arg name="script_filename" default=""/>
-  <xacro:arg name="input_recipe_filename" default=""/>
-  <xacro:arg name="output_recipe_filename" default=""/>
-  <xacro:arg name="include_thing1" default="true"/>
-  <xacro:arg name="include_thing2" default="true"/>
-  <xacro:arg name="thing1_robot_ip" default="192.168.50.19"/>
-  <xacro:arg name="thing1_wrist_camera_model" default=""/>
-  <xacro:arg name="thing1_joint_limits_parameters_file" default="$(find ur_description)/config/ur5/joint_limits.yaml"/>
-  <xacro:arg name="thing1_kinematics_parameters_file" default="$(find ur_description)/config/ur5/default_kinematics.yaml"/>
-  <xacro:arg name="thing1_physical_parameters_file" default="$(find ur_description)/config/ur5/physical_parameters.yaml"/>
-  <xacro:arg name="thing1_visual_parameters_file" default="$(find ur_description)/config/ur5/visual_parameters.yaml"/>
-  <xacro:arg name="thing2_robot_ip" default="192.168.50.20"/>
-  <xacro:arg name="thing2_wrist_camera_model" default=""/>
-  <xacro:arg name="thing2_joint_limits_parameters_file" default="$(find ur_description)/config/ur5/joint_limits.yaml"/>
-  <xacro:arg name="thing2_kinematics_parameters_file" default="$(find ur_description)/config/ur5/default_kinematics.yaml"/>
-  <xacro:arg name="thing2_physical_parameters_file" default="$(find ur_description)/config/ur5/physical_parameters.yaml"/>
-  <xacro:arg name="thing2_visual_parameters_file" default="$(find ur_description)/config/ur5/visual_parameters.yaml"/>
+  <xacro:include
+        filename="$(find ur5_workbench_description)/urdf/ur5_workbench_macro.xacro"
+    />
+  <xacro:arg name="include_ros2_control" default="false" />
+  <xacro:arg name="script_filename" default="" />
+  <xacro:arg name="input_recipe_filename" default="" />
+  <xacro:arg name="output_recipe_filename" default="" />
+  <xacro:arg name="include_thing1" default="true" />
+  <xacro:arg name="include_thing2" default="true" />
+  <xacro:arg name="thing1_use_gripper" default="true" />
+  <xacro:arg name="thing1_gripper_com_port" default="/dev/ttyUSB3" />
+  <xacro:arg name="thing1_use_fts" default="true" />
+  <xacro:arg name="thing1_fts_dev" default="ttyUSB0" />
+  <xacro:arg name="thing1_robot_ip" default="192.168.50.19" />
+  <xacro:arg name="thing1_wrist_camera_model" default="" />
+  <xacro:arg
+        name="thing1_joint_limits_parameters_file"
+        default="$(find ur_description)/config/ur5/joint_limits.yaml"
+    />
+  <xacro:arg
+        name="thing1_kinematics_parameters_file"
+        default="$(find ur_description)/config/ur5/default_kinematics.yaml"
+    />
+  <xacro:arg
+        name="thing1_physical_parameters_file"
+        default="$(find ur_description)/config/ur5/physical_parameters.yaml"
+    />
+  <xacro:arg
+        name="thing1_visual_parameters_file"
+        default="$(find ur_description)/config/ur5/visual_parameters.yaml"
+    />
+  <xacro:arg name="thing2_use_gripper" default="true" />
+  <xacro:arg name="thing2_gripper_com_port" default="/dev/ttyUSB2" />
+  <xacro:arg name="thing2_use_fts" default="true" />
+  <xacro:arg name="thing2_fts_dev" default="ttyUSB1" />
+  <xacro:arg name="thing2_robot_ip" default="192.168.50.20" />
+  <xacro:arg name="thing2_wrist_camera_model" default="" />
+  <xacro:arg
+        name="thing2_joint_limits_parameters_file"
+        default="$(find ur_description)/config/ur5/joint_limits.yaml"
+    />
+  <xacro:arg
+        name="thing2_kinematics_parameters_file"
+        default="$(find ur_description)/config/ur5/default_kinematics.yaml"
+    />
+  <xacro:arg
+        name="thing2_physical_parameters_file"
+        default="$(find ur_description)/config/ur5/physical_parameters.yaml"
+    />
+  <xacro:arg
+        name="thing2_visual_parameters_file"
+        default="$(find ur_description)/config/ur5/visual_parameters.yaml"
+    />
   <link name="world" />
   <xacro:ur5_workbench
-    parent="world"
-    include_ros2_control="$(arg include_ros2_control)"
-    script_filename="$(arg script_filename)"
-    input_recipe_filename="$(arg input_recipe_filename)"
-    output_recipe_filename="$(arg output_recipe_filename)"
-    include_thing1="$(arg include_thing1)"
-    include_thing2="$(arg include_thing2)"
-    thing1_robot_ip="$(arg thing1_robot_ip)"
-    thing1_wrist_camera_model="$(arg thing1_wrist_camera_model)"
-    thing1_joint_limits_parameters_file="$(arg thing1_joint_limits_parameters_file)"
-    thing1_kinematics_parameters_file="$(arg thing1_kinematics_parameters_file)"
-    thing1_physical_parameters_file="$(arg thing1_physical_parameters_file)"
-    thing1_visual_parameters_file="$(arg thing1_visual_parameters_file)"
-    thing2_robot_ip="$(arg thing2_robot_ip)"
-    thing2_wrist_camera_model="$(arg thing2_wrist_camera_model)"
-    thing2_joint_limits_parameters_file="$(arg thing2_joint_limits_parameters_file)"
-    thing2_kinematics_parameters_file="$(arg thing2_kinematics_parameters_file)"
-    thing2_physical_parameters_file="$(arg thing2_physical_parameters_file)"
-    thing2_visual_parameters_file="$(arg thing2_visual_parameters_file)"
-  >
+        parent="world"
+        include_ros2_control="$(arg include_ros2_control)"
+        script_filename="$(arg script_filename)"
+        input_recipe_filename="$(arg input_recipe_filename)"
+        output_recipe_filename="$(arg output_recipe_filename)"
+        include_thing1="$(arg include_thing1)"
+        include_thing2="$(arg include_thing2)"
+        thing1_use_gripper="$(arg thing1_use_gripper)"
+        thing1_gripper_com_port="$(arg thing1_gripper_com_port)"
+        thing1_use_fts="$(arg thing1_use_fts)"
+        thing1_fts_dev="$(arg thing1_fts_dev)"
+        thing1_robot_ip="$(arg thing1_robot_ip)"
+        thing1_wrist_camera_model="$(arg thing1_wrist_camera_model)"
+        thing1_joint_limits_parameters_file="$(arg thing1_joint_limits_parameters_file)"
+        thing1_kinematics_parameters_file="$(arg thing1_kinematics_parameters_file)"
+        thing1_physical_parameters_file="$(arg thing1_physical_parameters_file)"
+        thing1_visual_parameters_file="$(arg thing1_visual_parameters_file)"
+        thing2_gripper_com_port="$(arg thing2_gripper_com_port)"
+        thing2_use_gripper="$(arg thing2_use_gripper)"
+        thing2_use_fts="$(arg thing2_use_fts)"
+        thing2_fts_dev="$(arg thing2_fts_dev)"
+        thing2_robot_ip="$(arg thing2_robot_ip)"
+        thing2_wrist_camera_model="$(arg thing2_wrist_camera_model)"
+        thing2_joint_limits_parameters_file="$(arg thing2_joint_limits_parameters_file)"
+        thing2_kinematics_parameters_file="$(arg thing2_kinematics_parameters_file)"
+        thing2_physical_parameters_file="$(arg thing2_physical_parameters_file)"
+        thing2_visual_parameters_file="$(arg thing2_visual_parameters_file)"
+    >
     <origin xyz="0 0 0" rpy="0 0 0" />
   </xacro:ur5_workbench>

File: src/ur5_workbench_description/urdf/ur5_workbench_macro.xacro (robot description, xacro)
@@ -1,10 +1,14 @@
 <?xml version="1.0" ?>
 <robot xmlns:xacro="http://www.ros.org/wiki/xacro">
-  <xacro:include filename="$(find ur5_workbench_description)/urdf/thing_macro.xacro" />
+  <xacro:include
+        filename="$(find ur5_workbench_description)/urdf/thing_macro.xacro"
+    />
   <xacro:macro
-    name="ur5_workbench"
-    params="
+        name="ur5_workbench"
+        params="
       parent
       *origin
+      static_camera_model:=''
+      static_camera_extrinsics_file:=''
       include_ros2_control:=false
       script_filename:=''
@@ -18,4 +22,8 @@
       thing1_visual_parameters_file
       thing1_robot_ip:=192.168.50.19
+      thing1_fts_dev:=ttyUSB0
+      thing1_use_fts:=true
+      thing1_gripper_com_port:='/dev/ttyUSB3'
+      thing1_use_gripper:=true
       include_thing2:=true
       thing2_wrist_camera_model:=''
@@ -25,6 +33,10 @@
       thing2_visual_parameters_file
       thing2_robot_ip:=192.168.50.20
+      thing2_fts_dev:=ttyUSB1
+      thing2_use_fts:=true
+      thing2_gripper_com_port:='/dev/ttyUSB2'
+      thing2_use_gripper:=true
       "
-  >
+    >
     <joint name="table_joint" type="fixed">
       <xacro:insert_block name="origin" />
@@ -35,13 +47,21 @@
     <xacro:if value="${include_thing1}">
       <xacro:thing
-        name="thing1"
-        parent="table"
-        include_ros2_control="${include_ros2_control}"
-        wrist_camera_model="${thing1_wrist_camera_model}"
-        joint_limits_parameters_file="${thing1_joint_limits_parameters_file}"
-        kinematics_parameters_file="${thing1_kinematics_parameters_file}"
-        physical_parameters_file="${thing1_physical_parameters_file}"
-        visual_parameters_file="${thing1_visual_parameters_file}"
-      >
+                name="thing1"
+                parent="table"
+                include_ros2_control="${include_ros2_control}"
+                robot_ip="${thing1_robot_ip}"
+                script_filename="${script_filename}"
+                input_recipe_filename="${input_recipe_filename}"
+                output_recipe_filename="${output_recipe_filename}"
+                wrist_camera_model="${thing1_wrist_camera_model}"
+                joint_limits_parameters_file="${thing1_joint_limits_parameters_file}"
+                kinematics_parameters_file="${thing1_kinematics_parameters_file}"
+                physical_parameters_file="${thing1_physical_parameters_file}"
+                visual_parameters_file="${thing1_visual_parameters_file}"
+                fts_dev="${thing1_fts_dev}"
+                use_fts="${thing1_use_fts}"
+                gripper_com_port="${thing1_gripper_com_port}"
+                use_gripper="${thing1_use_gripper}"
+            >
         <origin xyz="1.905 0.381 0" rpy="0 0 ${pi/2}" />
       </xacro:thing>
@@ -49,16 +69,26 @@
     <xacro:if value="${include_thing2}">
       <xacro:thing
-        name="thing2"
-        parent="table"
-        include_ros2_control="${include_ros2_control}"
-        wrist_camera_model="${thing2_wrist_camera_model}"
-        joint_limits_parameters_file="${thing2_joint_limits_parameters_file}"
-        kinematics_parameters_file="${thing2_kinematics_parameters_file}"
-        physical_parameters_file="${thing2_physical_parameters_file}"
-        visual_parameters_file="${thing2_visual_parameters_file}"
-      >
+                name="thing2"
+                parent="table"
+                include_ros2_control="${include_ros2_control}"
+                robot_ip="${thing2_robot_ip}"
+                script_filename="${script_filename}"
+                input_recipe_filename="${input_recipe_filename}"
+                output_recipe_filename="${output_recipe_filename}"
+                wrist_camera_model="${thing2_wrist_camera_model}"
+                joint_limits_parameters_file="${thing2_joint_limits_parameters_file}"
+                kinematics_parameters_file="${thing2_kinematics_parameters_file}"
+                physical_parameters_file="${thing2_physical_parameters_file}"
+                visual_parameters_file="${thing2_visual_parameters_file}"
+                fts_dev="${thing2_fts_dev}"
+                use_fts="${thing2_use_fts}"
+                gripper_com_port="${thing2_gripper_com_port}"
+                use_gripper="${thing2_use_gripper}"
+            >
         <origin xyz="0.381 0.381 0" rpy="0 0 ${pi/2}" />
       </xacro:thing>
     </xacro:if>
+    <xacro:if value="${static_camera_model != ''}">
+    </xacro:if>
   </xacro:macro>
 </robot>
