Commit message: Added wrist camera support, made progress on ur ros driver, made mujoco config urdf parameterizable

File: mjcf_data/robot_description_formatted.urdf (robot description, URDF)
Before this commit: robot ur5_workbench, 51 links, 50 joints
Links:
- removed link falling_box
- added link thing2_camera_link, mass 1e-9
- added link thing2_camera_mount_link, mass 1e-09; visual mesh filename=full/camera_mount.stl
- added link thing2_d405_bottom_screw_frame
- added link thing2_d405_link, mass 0.072; visual mesh filename=full/d405.stl scale=0.001 0.001 0.001
- added link thing2_tool_link, mass 1e-9
- added link thing2_wrist_camera_frame
Joints:
- removed joint falling_box_joint
- added joint thing2_camera_link_frame: type fixed, parent thing2_camera_mount_link, child thing2_camera_link, origin xyz=-8.05759e-05 -0.0777769 0.00836815 rpy=-0.139625 3.04604e-07 -4.28088e-08, axis 0 0 0
- added joint thing2_camera_mount_joint: type fixed, parent thing2_robotiq_ft_frame_id, child thing2_camera_mount_link, origin xyz=0 0 0 rpy=0 0 0
- added joint thing2_d405_joint: type fixed, parent thing2_camera_link, child thing2_d405_bottom_screw_frame, origin xyz=0 0.021 0.009 rpy=0 -1.5707963267948966 1.5707963267948966
- added joint thing2_d405_link_joint: type fixed, parent thing2_d405_bottom_screw_frame, child thing2_d405_link, origin xyz=0.01085 0.009 0.021 rpy=0 0 0
- added joint thing2_tool_link_frame: type fixed, parent thing2_camera_mount_link, child thing2_tool_link, origin xyz=0 0 0.00299997 rpy=0 0 0, axis 0 0 0
- added joint thing2_wrist_camera_frame_joint: type fixed, parent thing2_d405_link, child thing2_wrist_camera_frame, origin xyz=0 0 0 rpy=-1.5707963267948966 0 -1.5707963267948966
- joint thing2_robotiq_85_base_joint: parent thing2_robotiq_ft_frame_id -> thing2_tool_link

File: src/ur5_workbench_description/urdf/thing_macro.xacro (robot description, xacro)
@@ -6,9 +6,10 @@
   <xacro:include filename="$(find robotiq_ft_sensor_description)/urdf/robotiq_fts.ros2_control.xacro" />
   <xacro:include filename="$(find ur5_workbench_description)/urdf/camera_mount_macro.xacro" />
+  <xacro:include filename="$(find ur_robot_driver)/urdf/ur.ros2_control.xacro" />
   <xacro:macro name="thing" params="
     name
     parent
     *origin
-    include_ros2_control:=true
+    include_ros2_control:=false
     wrist_camera_model:=''
     joint_limits_parameters_file
@@ -16,4 +17,9 @@
     physical_parameters_file
     visual_parameters_file
+    robot_ip:=''
+    script_filename:=''
+    input_recipe_filename:=''
+    output_recipe_filename:=''
+    initial_positions:=${dict(shoulder_pan_joint=0.0,shoulder_lift_joint=-1.57,elbow_joint=0.0,wrist_1_joint=-1.57,wrist_2_joint=0.0,wrist_3_joint=0.0)}
   ">
     <xacro:ur_robot
@@ -31,10 +37,4 @@
       <origin xyz="0 0 -0.004" rpy="0 0 ${-pi/2}" />
     </xacro:robotiq_ft300>
-    <xacro:if value="${include_ros2_control}">
-      <xacro:robotiq_fts_ros2_control
-        name="${name}_"
-        tf_prefix="${name}_"
-      />
-    </xacro:if>
     <xacro:if value="${wrist_camera_model != ''}">
       <xacro:include filename="$(find realsense2_description)/urdf/_${wrist_camera_model}.urdf.xacro" />
@@ -67,4 +67,21 @@
       </xacro:robotiq_gripper>
     </xacro:unless>
+    <!-- ros2_control macros -->
+    <xacro:if value="${include_ros2_control}">
+      <xacro:robotiq_fts_ros2_control
+        name="${name}_"
+        tf_prefix="${name}_"
+      />
+      <xacro:ur_ros2_control
+        name="${name}_"
+        tf_prefix="${name}_"
+        kinematics_parameters_file="${kinematics_parameters_file}"
+        robot_ip="${robot_ip}"
+        script_filename="${script_filename}"
+        input_recipe_filename="${input_recipe_filename}"
+        output_recipe_filename="${output_recipe_filename}"
+        initial_positions="${initial_positions}"
+      />
+    </xacro:if>
   </xacro:macro>
 </robot>

File: src/ur5_workbench_description/urdf/ur5_workbench.urdf.xacro (robot description, xacro)
@@ -2,7 +2,11 @@
 <robot name="ur5_workbench" xmlns:xacro="http://www.ros.org/wiki/xacro">
   <xacro:include filename="$(find ur5_workbench_description)/urdf/ur5_workbench_macro.xacro" />
-  <xacro:arg name="include_ros2_control" default="true"/>
+  <xacro:arg name="include_ros2_control" default="false"/>
+  <xacro:arg name="script_filename" default=""/>
+  <xacro:arg name="input_recipe_filename" default=""/>
+  <xacro:arg name="output_recipe_filename" default=""/>
   <xacro:arg name="include_thing1" default="true"/>
   <xacro:arg name="include_thing2" default="true"/>
+  <xacro:arg name="thing1_robot_ip" default=""/>
   <xacro:arg name="thing1_wrist_camera_model" default=""/>
   <xacro:arg name="thing1_joint_limits_parameters_file" default="$(find ur_description)/config/ur5/joint_limits.yaml"/>
@@ -10,4 +14,5 @@
   <xacro:arg name="thing1_physical_parameters_file" default="$(find ur_description)/config/ur5/physical_parameters.yaml"/>
   <xacro:arg name="thing1_visual_parameters_file" default="$(find ur_description)/config/ur5/visual_parameters.yaml"/>
+  <xacro:arg name="thing2_robot_ip" default=""/>
   <xacro:arg name="thing2_wrist_camera_model" default=""/>
   <xacro:arg name="thing2_joint_limits_parameters_file" default="$(find ur_description)/config/ur5/joint_limits.yaml"/>
@@ -19,6 +24,10 @@
     parent="world"
     include_ros2_control="$(arg include_ros2_control)"
+    script_filename="$(arg script_filename)"
+    input_recipe_filename="$(arg input_recipe_filename)"
+    output_recipe_filename="$(arg output_recipe_filename)"
     include_thing1="$(arg include_thing1)"
     include_thing2="$(arg include_thing2)"
+    thing1_robot_ip="$(arg thing1_robot_ip)"
     thing1_wrist_camera_model="$(arg thing1_wrist_camera_model)"
     thing1_joint_limits_parameters_file="$(arg thing1_joint_limits_parameters_file)"
@@ -26,4 +35,5 @@
     thing1_physical_parameters_file="$(arg thing1_physical_parameters_file)"
     thing1_visual_parameters_file="$(arg thing1_visual_parameters_file)"
+    thing2_robot_ip="$(arg thing2_robot_ip)"
     thing2_wrist_camera_model="$(arg thing2_wrist_camera_model)"
     thing2_joint_limits_parameters_file="$(arg thing2_joint_limits_parameters_file)"

File: src/ur5_workbench_description/urdf/ur5_workbench_macro.xacro (robot description, xacro)
@@ -7,5 +7,8 @@
       parent
       *origin
-      include_ros2_control:=true
+      include_ros2_control:=false
+      script_filename:=''
+      input_recipe_filename:=''
+      output_recipe_filename:=''
       include_thing1:=true
       thing1_wrist_camera_model:=''
@@ -14,4 +17,5 @@
       thing1_physical_parameters_file
       thing1_visual_parameters_file
+      thing1_robot_ip:=''
       include_thing2:=true
       thing2_wrist_camera_model:=''
@@ -20,4 +24,5 @@
       thing2_physical_parameters_file
       thing2_visual_parameters_file
+      thing2_robot_ip:=''
       "
   >

File: src/ur5_workbench_mujoco_config/urdf/ur5_workbench.mujoco_ros2_control.xacro (robot description, xacro)
@@ -4,4 +4,9 @@
     filename="$(find ur5_workbench_description)/urdf/ur5_workbench_macro.xacro"
   />
+  <xacro:arg name="include_thing1" default="true" />
+  <xacro:arg name="include_thing2" default="true" />
+  <xacro:arg
+    name="thing1_wrist_camera_model"
+    default="" />
   <xacro:arg
     name="thing1_joint_limits_parameters_file"
@@ -20,4 +25,7 @@
     default="$(find ur_description)/config/ur5/visual_parameters.yaml"
   />
+  <xacro:arg
+    name="thing2_wrist_camera_model"
+    default="" />
   <xacro:arg
     name="thing2_joint_limits_parameters_file"
@@ -40,8 +48,12 @@
     parent="world"
     include_ros2_control="false"
+    include_thing1="$(arg include_thing1)"
+    include_thing2="$(arg include_thing2)"
+    thing1_wrist_camera_model="$(arg thing1_wrist_camera_model)"
     thing1_joint_limits_parameters_file="$(arg thing1_joint_limits_parameters_file)"
     thing1_kinematics_parameters_file="$(arg thing1_kinematics_parameters_file)"
     thing1_physical_parameters_file="$(arg thing1_physical_parameters_file)"
     thing1_visual_parameters_file="$(arg thing1_visual_parameters_file)"
+    thing2_wrist_camera_model="$(arg thing2_wrist_camera_model)"
     thing2_joint_limits_parameters_file="$(arg thing2_joint_limits_parameters_file)"
     thing2_kinematics_parameters_file="$(arg thing2_kinematics_parameters_file)"
@@ -136,4 +148,5 @@
       </default>
       <actuator>
+      <xacro:if value="$(arg include_thing1)">
         <position
           class="size4"
@@ -167,4 +180,6 @@
         />
         <position tendon="thing1_split" name="thing1_robotiq_85_left_knuckle_joint" kp="10000" dampratio="1.0" ctrlrange="0.0 0.79" forcerange="-150 150"/>
+      </xacro:if>
+      <xacro:if value="$(arg include_thing2)">
         <position
           class="size4"
@@ -198,16 +213,22 @@
         />
         <position tendon="thing2_split" name="thing2_robotiq_85_left_knuckle_joint" kp="10000" dampratio="1.0" ctrlrange="0.0 0.79" forcerange="-150 150"/>
+        </xacro:if>
       </actuator>
       <tendon>
+        <xacro:if value="$(arg include_thing1)">
         <fixed name="thing1_split">
           <joint joint="thing1_robotiq_85_left_knuckle_joint" coef="0.5"/>
           <joint joint="thing1_robotiq_85_right_knuckle_joint" coef="-0.5"/>
         </fixed>
+        </xacro:if>
+        <xacro:if value="$(arg include_thing2)">
         <fixed name="thing2_split">
           <joint joint="thing2_robotiq_85_left_knuckle_joint" coef="0.5"/>
           <joint joint="thing2_robotiq_85_right_knuckle_joint" coef="-0.5"/>
         </fixed>
+        </xacro:if>
       </tendon>
       <contact>
+        <xacro:if value="$(arg include_thing1)">
         <exclude body1="world" body2="thing1_shoulder_link" />
         <exclude
@@ -244,4 +265,6 @@
         />
         <exclude body1="thing1_robotiq_85_left_finger_tip_link" body2="thing1_robotiq_85_right_finger_tip_link" />
+        </xacro:if>
+        <xacro:if value="$(arg include_thing2)" >
         <exclude body1="world" body2="thing2_shoulder_link" />
         <exclude
@@ -278,13 +301,19 @@
         />
         <exclude body1="thing2_robotiq_85_left_finger_tip_link" body2="thing2_robotiq_85_right_finger_tip_link" />
+        </xacro:if>
       </contact>
       <equality>
-        <connect anchor="-0.0371575 0.0 0.043422" body1="thing1_robotiq_85_right_inner_knuckle_link" body2="thing1_robotiq_85_right_finger_tip_link" solimp="0.95 0.99 0.001" solref="0.005 1"/>
-        <connect anchor="0.0371575 0.0 0.043422" body1="thing1_robotiq_85_left_inner_knuckle_link" body2="thing1_robotiq_85_left_finger_tip_link" solimp="0.95 0.99 0.001" solref="0.005 1"/>
-        <joint joint1="thing1_robotiq_85_left_knuckle_joint" joint2="thing1_robotiq_85_right_knuckle_joint" polycoef="0 -1 0 0 0" solimp="0.95 0.99 0.001" solref="0.005 1"/>
-        <connect anchor="-0.0371575 0.0 0.043422" body1="thing2_robotiq_85_right_inner_knuckle_link" body2="thing2_robotiq_85_right_finger_tip_link" solimp="0.95 0.99 0.001" solref="0.005 1"/>
-        <connect anchor="0.0371575 0.0 0.043422" body1="thing2_robotiq_85_left_inner_knuckle_link" body2="thing2_robotiq_85_left_finger_tip_link" solimp="0.95 0.99 0.001" solref="0.005 1"/>
-        <joint joint1="thing2_robotiq_85_left_knuckle_joint" joint2="thing2_robotiq_85_right_knuckle_joint" polycoef="0 -1 0 0 0" solimp="0.95 0.99 0.001" solref="0.005 1"/>
+        <xacro:if value="$(arg include_thing1)" >
+          <connect anchor="-0.0371575 0.0 0.043422" body1="thing1_robotiq_85_right_inner_knuckle_link" body2="thing1_robotiq_85_right_finger_tip_link" solimp="0.95 0.99 0.001" solref="0.005 1"/>
+          <connect anchor="0.0371575 0.0 0.043422" body1="thing1_robotiq_85_left_inner_knuckle_link" body2="thing1_robotiq_85_left_finger_tip_link" solimp="0.95 0.99 0.001" solref="0.005 1"/>
+          <joint joint1="thing1_robotiq_85_left_knuckle_joint" joint2="thing1_robotiq_85_right_knuckle_joint" polycoef="0 -1 0 0 0" solimp="0.95 0.99 0.001" solref="0.005 1"/>
+        </xacro:if>
+        <xacro:if value="$(arg include_thing2)" >
+          <connect anchor="-0.0371575 0.0 0.043422" body1="thing2_robotiq_85_right_inner_knuckle_link" body2="thing2_robotiq_85_right_finger_tip_link" solimp="0.95 0.99 0.001" solref="0.005 1"/>
+          <connect anchor="0.0371575 0.0 0.043422" body1="thing2_robotiq_85_left_inner_knuckle_link" body2="thing2_robotiq_85_left_finger_tip_link" solimp="0.95 0.99 0.001" solref="0.005 1"/>
+          <joint joint1="thing2_robotiq_85_left_knuckle_joint" joint2="thing2_robotiq_85_right_knuckle_joint" polycoef="0 -1 0 0 0" solimp="0.95 0.99 0.001" solref="0.005 1"/>
+        </xacro:if>
       </equality>
+      <xacro:if value="$(arg include_thing1)" >
       <sensor>
         <force
@@ -297,4 +326,6 @@
         />
       </sensor>
+      </xacro:if>
+      <xacro:if value="$(arg include_thing2)" >
       <sensor>
         <force
@@ -307,13 +338,24 @@
         />
       </sensor>
+      </xacro:if>
     </raw_inputs>
     <processed_inputs>
-      <modify_element type="joint" name="thing1_robotiq_85_left_knuckle_joint" armature="0.5" frictionloss="5.0" />
-      <modify_element type="joint" name="thing1_robotiq_85_right_knuckle_joint" armature="0.5" frictionloss="5.0" />
-      <modify_element type="joint" name="thing2_robotiq_85_left_knuckle_joint" armature="0.5" frictionloss="5.0" />
-      <modify_element type="joint" name="thing2_robotiq_85_right_knuckle_joint" armature="0.5" frictionloss="5.0" />
+      <xacro:if value="$(arg include_thing1)" >
+        <xacro:if value="${'$(arg thing1_wrist_camera_model)' != ''}">
+          <camera name="thing1_wrist_camera" site="thing1_wrist_camera_frame" mode="fixed" fovy="45" resolution="640 480" />
+        </xacro:if>
+        <modify_element type="joint" name="thing1_robotiq_85_left_knuckle_joint" armature="0.5" frictionloss="5.0" />
+        <modify_element type="joint" name="thing1_robotiq_85_right_knuckle_joint" armature="0.5" frictionloss="5.0" />
+      </xacro:if>
+      <xacro:if value="$(arg include_thing2)" >
+        <xacro:if value="${'$(arg thing2_wrist_camera_model)' != ''}">
+          <camera name="thing2_wrist_camera" site="thing2_wrist_camera_frame" mode="fixed" fovy="45" resolution="640 480" />
+        </xacro:if>
+        <modify_element type="joint" name="thing2_robotiq_85_left_knuckle_joint" armature="0.5" frictionloss="5.0" />
+        <modify_element type="joint" name="thing2_robotiq_85_right_knuckle_joint" armature="0.5" frictionloss="5.0" />
+      </xacro:if>
     </processed_inputs>
   </mujoco_inputs>
-  <joint name="falling_box_joint" type="floating">
+  <!-- <joint name="falling_box_joint" type="floating">
     <origin xyz="0 0 0" rpy="0 0 0" />
     <parent link="world" />
@@ -335,5 +377,25 @@
       </geometry>
     </collision>
-  </link>
+  </link> -->
+  <xacro:if value="$(arg include_thing1)">
+    <xacro:if value="${'$(arg thing1_wrist_camera_model)' != ''}">
+      <joint name="thing1_wrist_camera_frame_joint" type="fixed">
+        <origin xyz="0 0 0" rpy="-${pi/2} 0 -${pi/2}" />
+        <parent link="thing1_$(arg thing1_wrist_camera_model)_link" />
+        <child link="thing1_wrist_camera_frame" />
+      </joint>
+      <link name="thing1_wrist_camera_frame" />
+    </xacro:if>
+  </xacro:if>
+  <xacro:if value="$(arg include_thing2)">
+    <xacro:if value="${'$(arg thing2_wrist_camera_model)' != ''}">
+      <joint name="thing2_wrist_camera_frame_joint" type="fixed">
+        <origin xyz="0 0 0" rpy="-${pi/2} 0 -${pi/2}" />
+        <parent link="thing2_$(arg thing2_wrist_camera_model)_link" />
+        <child link="thing2_wrist_camera_frame" />
+      </joint>
+      <link name="thing2_wrist_camera_frame" />
+    </xacro:if>
+  </xacro:if>
   <ros2_control name="MujocoSystem" type="system">
     <hardware>
@@ -341,7 +403,26 @@
       <param name="sim_speed_factor">1.0</param>
     </hardware>
-    <xacro:mujoco_ur5 prefix="thing1_" />
-    <xacro:mujoco_ur5 prefix="thing2_" />
-    <joint name="falling_box_joint" />
+    <xacro:if value="$(arg include_thing1)">
+      <xacro:if value="${'$(arg thing1_wrist_camera_model)' != ''}">
+        <sensor name="thing1_wrist_camera">
+          <param name="frame_name">thing1_wrist_camera_frame</param>
+          <param name="info_topic">/thing1_wrist_camera/color/camera_info</param>
+          <param name="image_topic">/thing1_wrist_camera/color/image_raw</param>
+          <param name="depth_topic">/thing1_wrist_camera/aligned_depth_to_color/image_raw</param>
+        </sensor>
+      </xacro:if>
+      <xacro:mujoco_ur5 prefix="thing1_" />
+    </xacro:if>
+    <xacro:if value="$(arg include_thing2)">
+      <xacro:if value="${'$(arg thing2_wrist_camera_model)' != ''}">
+        <sensor name="thing2_wrist_camera">
+          <param name="frame_name">thing2_wrist_camera_frame</param>
+          <param name="info_topic">/thing2_wrist_camera/color/camera_info</param>
+          <param name="image_topic">/thing2_wrist_camera/color/image_raw</param>
+          <param name="depth_topic">/thing2_wrist_camera/aligned_depth_to_color/image_raw</param>
+        </sensor>
+      </xacro:if>
+      <xacro:mujoco_ur5 prefix="thing2_" />
+    </xacro:if>
   </ros2_control>
 </robot>

Commit message: Removed unnecessary moveit launches and consolidated into one launch

File: mjcf_data/robot_description_formatted.urdf (robot description, URDF)
Before this commit: robot ur5_workbench, 56 links, 55 joints
Links:
- removed link thing2_camera_link
- removed link thing2_camera_mount_link
- removed link thing2_d405_bottom_screw_frame
- removed link thing2_d405_link
- removed link thing2_tool_link
- removed link thing2_wrist_camera_frame
- added link thing1_tcp_frame
- added link thing2_tcp_frame
Joints:
- removed joint thing2_camera_link_frame
- removed joint thing2_camera_mount_joint
- removed joint thing2_d405_joint
- removed joint thing2_d405_link_joint
- removed joint thing2_tool_link_frame
- removed joint thing2_wrist_camera_frame_joint
- added joint thing1_tcp_joint: type fixed, parent thing1_robotiq_85_base_link, child thing1_tcp_frame, origin xyz=0 0 0.135 rpy=0 0 0
- added joint thing2_tcp_joint: type fixed, parent thing2_robotiq_85_base_link, child thing2_tcp_frame, origin xyz=0 0 0.135 rpy=0 0 0
- joint thing2_robotiq_85_base_joint: parent thing2_tool_link -> thing2_robotiq_ft_frame_id
